File: IS42S16160.kicad_sch (KiCad schematic)
At the start: 8 parts, among them U2 IS42S16160J-6BLI

Commit message: 98% finished, st-link part left
Other:
- note added: "PC2"
- note added: "PC3"
- note added: "PD0"
- note added: "PD1"
- note added: "PD10"
- note added: "PD14"
- note added: "PD15"
- note added: "PD8"
- note added: "PD9"
- note added: "PE0"
- note added: "PE1"
- note added: "PE10"
- note added: "PE11"
- note added: "PE12"
- note added: "PE13"
- note added: "PE14"
- note added: "PE15"
- note added: "PE7"
- note added: "PE8"
- note added: "PE9"
- note added: "PF0"
- note added: "PF1"
- note added: "PF11"
- note added: "PF12"
- note added: "PF13"
- note added: "PF14"
- note added: "PF15"
- note added: "PF2"
- note added: "PF3"
- note added: "PF4"
- note added: "PF5"
- note added: "PG0"
- note added: "PG1"
- note added: "PG15"
- note added: "PG2"
- note added: "PG4"
- note added: "PG5"
- note added: "PG8"
- note added: "PH5"

Commit message: Adding JLCPCB Part #
Parts:
- C26, C27, C28, C29, C30, C32, C33: JLCPCB Part # (none) -> C307380
- U2: JLCPCB Part # (none) -> C1348766
Changed lines of the file:
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@@
+			)
+		)
+		(property "JLCPCB Part #" "C307380"
+			(at 120.65 132.08 0)
+			(effects
+				(font
+					(size 1.27 1.27)
+				)
+				(hide yes)
 			)
 		)
@@
 			)
 		)
+		(property "JLCPCB Part #" "C307380"
+			(at 120.65 124.46 0)
+			(effects
+				(font
+					(size 1.27 1.27)
+				)
+				(hide yes)
+			)
+		)
 		(pin "1"
 		)
@@
 		)
 		(property "Description" "Unpolarized capacitor, small symbol"
+			(at 120.65 119.38 0)
+			(effects
+				(font
+					(size 1.27 1.27)
+				)
+				(hide yes)
+			)
+		)
+		(property "JLCPCB Part #" "C307380"
 			(at 120.65 119.38 0)
 			(effects
@@
 			)
 		)
+		(property "JLCPCB Part #" "C1348766"
+			(at 142.24 93.98 0)
+			(effects
+				(font
+					(size 1.27 1.27)
+				)
+				(hide yes)
+			)
+		)
 		(pin "C7"
 		)
@@
 			)
 		)
+		(property "JLCPCB Part #" "C307380"
+			(at 113.03 134.62 0)
+			(effects
+				(font
+					(size 1.27 1.27)
+				)
+				(hide yes)
+			)
+		)
 		(pin "1"
 		)
@@
 		)
 		(property "Description" "Unpolarized capacitor, small symbol"
+			(at 113.03 127 0)
+			(effects
+				(font
+					(size 1.27 1.27)
+				)
+				(hide yes)
+			)
+		)
+		(property "JLCPCB Part #" "C307380"
 			(at 113.03 127 0)
 			(effects
@@
 			)
 		)
+		(property "JLCPCB Part #" "C307380"
+			(at 120.65 137.16 0)
+			(effects
+				(font
+					(size 1.27 1.27)
+				)
+				(hide yes)
+			)
+		)
 		(pin "1"
 		)
@@
 			(at 113.03 121.92 0)
 			(effects
+				(font
+					(size 1.27 1.27)
+				)
+				(hide yes)
+			)
+		)
+		(property "JLCPCB Part #" "C307380"
+			(at 113.03 121.92 0)
+			(effects
