File: MT25QL256.kicad_sch (KiCad schematic)
At the start: 7 parts, among them U3 W25Q32JVZP, U5 W25Q32JVZP

Commit message: SDRAM finished, changed castellated to 23pin each side, few pins unconnected
Parts:
- U3, U5: footprint Package_SON:WSON-8-1EP_8x6mm_P1.27mm_EP3.4x4.3mm -> W25Q256JVEIQ:SON127P800X600X80-9N
Changed lines of the file:
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@@
 			)
 		)
-		(property "Footprint" "Package_SON:WSON-8-1EP_8x6mm_P1.27mm_EP3.4x4.3mm"
+		(property "Footprint" "W25Q256JVEIQ:SON127P800X600X80-9N"
 			(at 143.51 124.46 0)
 			(effects
@@
 			)
 		)
-		(property "Footprint" "Package_SON:WSON-8-1EP_8x6mm_P1.27mm_EP3.4x4.3mm"
+		(property "Footprint" "W25Q256JVEIQ:SON127P800X600X80-9N"
 			(at 143.51 73.66 0)
 			(effects
